Commit message: Xacro Configuration

File: src/my_bot/description/robot.urdf.xacro (robot description, xacro)
@@ -1,4 +1,4 @@
 <?xml version="1.0"?>
 <robot xmlns:xacro="http://www.ros.org/wiki/xacro"  name="robot">
-    <xacro:include filename = "robot_core.xacro" />
+    <xacro:include filename = "robot_core.xacro"/>
 </robot>

File: src/my_bot/description/robot_core.xacro (robot description, xacro)
@@ -1,3 +1,115 @@
 <?xml version="1.0"?>
 <robot xmlns:xacro="http://www.ros.org/wiki/xacro">
+    <material name="black">
+        <color rgba="0 0 0 1"/>
+    </material>
+    <material name="orange">
+        <color rgba="1 0.3 0.1 1"/>
+    </material>
+    <material name="blue">
+        <color rgba="0.2 0.2 1 1"/>
+    </material>
+    <material name="white">
+        <color rgba="1 1 1 1"/>
+    </material>
+    <!-- Base Link-->
+    <link name="base_link">
+    </link>
+    <!-- Chassis link -->
+    <joint name="chassis_joint" type="fixed">
+        <parent link="base_link"/>
+        <child link="chassis"/>
+        <origin xyz="0 0 0"/>
+    </joint>
+    <link name="chassis">
+        <visual>
+            <geometry>
+                <box size="0.255 0.19 0.045 "/>
+            </geometry>
+            <material name="white"/>
+        </visual>
+        <collision>
+            <geometry>
+                <box size="0.255 0.19 0.045 "/>
+            </geometry>
+        </collision>
+    </link>
+    <!-- front wheel -->
+    <joint name="front_left_wheel_joint" type="continuous">
+        <parent link="base_link"/>
+        <child link="front_left_wheel"/>
+        <origin xyz="0.1175 0.115 0" rpy="-${pi/2} 0 0"/>
+        <axis xyz="0 0 1"/>
+    </joint>
+    <link name="front_left_wheel">
+        <visual>
+            <geometry>
+                <cylinder radius="0.04" length="0.04"/>
+            </geometry>
+            <material name="blue"/>
+        </visual>
+        <collision>
+            <geometry>
+                <cylinder radius="0.04" length="0.04"/>
+            </geometry>
+        </collision>
+    </link>
+    <joint name="front_right_wheel_joint" type="continuous">
+        <parent link="base_link"/>
+        <child link="front_right_wheel"/>
+        <origin xyz="0.1175 -0.115 0" rpy="${pi/2} 0 0"/>
+        <axis xyz="0 0 1"/>
+    </joint>
+    <link name="front_right_wheel">
+        <visual>
+            <geometry>
+                <cylinder radius="0.04" length="0.04"/>
+            </geometry>
+            <material name="blue"/>
+        </visual>
+        <collision>
+            <geometry>
+                <cylinder radius="0.04" length="0.04"/>
+            </geometry>
+        </collision>
+    </link>
+    <!-- rear wheel -->
+    <joint name="rear_left_wheel_joint" type="continuous">
+        <parent link="base_link"/>
+        <child link="rear_left_wheel"/>
+        <origin xyz="-0.1175 0.115 0" rpy="-${pi/2} 0 0"/>
+        <axis xyz="0 0 1"/>
+    </joint>
+    <link name="rear_left_wheel">
+        <visual>
+            <geometry>
+                <cylinder radius="0.04" length="0.04"/>
+            </geometry>
+            <material name="blue"/>
+        </visual>
+        <collision>
+            <geometry>
+                <cylinder radius="0.04" length="0.04"/>
+            </geometry>
+        </collision>
+    </link>
+    <joint name="rear_right_wheel_joint" type="continuous">
+        <parent link="base_link"/>
+        <child link="rear_right_wheel"/>
+        <origin xyz="-0.1175 -0.115 0" rpy="${pi/2} 0 0"/>
+        <axis xyz="0 0 1"/>
+    </joint>
+    <link name="rear_right_wheel">
+        <visual>
+            <geometry>
+                <cylinder radius="0.04" length="0.04"/>
+            </geometry>
+            <material name="blue"/>
+        </visual>
+        <collision>
+            <geometry>
+                <cylinder radius="0.04" length="0.04"/>
+            </geometry>
+        </collision>
+    </link>
 </robot>

Commit message: Gazebo Configuration

File: src/my_bot/description/robot.urdf.xacro (robot description, xacro)
@@ -2,3 +2,4 @@
 <robot xmlns:xacro="http://www.ros.org/wiki/xacro"  name="robot">
     <xacro:include filename = "robot_core.xacro"/>
+    <xacro:include filename = "gazebo_control.xacro"/>
 </robot>

File: src/my_bot/description/robot_core.xacro (robot description, xacro)
@@ -1,14 +1,15 @@
 <?xml version="1.0"?>
 <robot xmlns:xacro="http://www.ros.org/wiki/xacro">
-    <material name="black">
+    <xacro:include filename="inertial_macros.xacro"/>
+    <material name="Black">
         <color rgba="0 0 0 1"/>
     </material>
-    <material name="orange">
+    <material name="Orange">
         <color rgba="1 0.3 0.1 1"/>
     </material>
-    <material name="blue">
+    <material name="Blue">
         <color rgba="0.2 0.2 1 1"/>
     </material>
-    <material name="white">
+    <material name="White">
         <color rgba="1 1 1 1"/>
     </material>
@@ -27,5 +28,5 @@
                 <box size="0.255 0.19 0.045 "/>
             </geometry>
-            <material name="white"/>
+            <material name="White"/>
         </visual>
         <collision>
@@ -34,5 +35,11 @@
             </geometry>
         </collision>
+        <xacro:inertial_box mass="0.5" x="0.255" y="0.19" z="0.045">
+            <origin xyz="0 0 0" rpy="0 0 0"/>
+        </xacro:inertial_box>
     </link>
+    <gazebo referece="chassis">
+        <material>Gazebo/White</material>
+    </gazebo>
     <!-- front wheel -->
     <joint name="front_left_wheel_joint" type="continuous">
@@ -47,5 +54,5 @@
                 <cylinder radius="0.04" length="0.04"/>
             </geometry>
-            <material name="blue"/>
+            <material name="Blue"/>
         </visual>
         <collision>
@@ -54,5 +61,11 @@
             </geometry>
         </collision>
+        <xacro:inertial_cylinder mass="0.1" length="0.04" radius="0.04">
+            <origin xyz="0 0 0" rpy="0 0 0"/>
+        </xacro:inertial_cylinder>
     </link>
+    <gazebo referece="front_left_wheel">
+        <material>Gazebo/Blue</material>
+    </gazebo>
     <joint name="front_right_wheel_joint" type="continuous">
         <parent link="base_link"/>
@@ -66,5 +79,5 @@
                 <cylinder radius="0.04" length="0.04"/>
             </geometry>
-            <material name="blue"/>
+            <material name="Blue"/>
         </visual>
         <collision>
@@ -73,5 +86,11 @@
             </geometry>
         </collision>
+        <xacro:inertial_cylinder mass="0.1" length="0.04" radius="0.04">
+            <origin xyz="0 0 0" rpy="0 0 0"/>
+        </xacro:inertial_cylinder>
     </link>
+    <gazebo referece="front_right_wheel">
+        <material>Gazebo/Blue</material>
+    </gazebo>
     <!-- rear wheel -->
     <joint name="rear_left_wheel_joint" type="continuous">
@@ -86,5 +105,5 @@
                 <cylinder radius="0.04" length="0.04"/>
             </geometry>
-            <material name="blue"/>
+            <material name="Blue"/>
         </visual>
         <collision>
@@ -93,5 +112,11 @@
             </geometry>
         </collision>
+        <xacro:inertial_cylinder mass="0.1" length="0.04" radius="0.04">
+            <origin xyz="0 0 0" rpy="0 0 0"/>
+        </xacro:inertial_cylinder>
     </link>
+    <gazebo referece="rear_left_wheel">
+        <material>Gazebo/Blue</material>
+    </gazebo>
     <joint name="rear_right_wheel_joint" type="continuous">
         <parent link="base_link"/>
@@ -105,5 +130,5 @@
                 <cylinder radius="0.04" length="0.04"/>
             </geometry>
-            <material name="blue"/>
+            <material name="Blue"/>
         </visual>
         <collision>
@@ -112,4 +137,10 @@
             </geometry>
         </collision>
+        <xacro:inertial_cylinder mass="0.1" length="0.04" radius="0.04">
+            <origin xyz="0 0 0" rpy="0 0 0"/>
+        </xacro:inertial_cylinder>
     </link>
+    <gazebo referece="rear_right_wheel">
+        <material>Gazebo/Blue</material>
+    </gazebo>
 </robot>
